File: Project/PCB/SWARMESH/SWARMESH.sch (EAGLE design)
At the start: 37 parts, among them IC1 4051N, IC2 L293D, Q1 TIP122, U1 ESP32DEVKITC

Commit message: updated name and deleted unnecessary components
Parts:
- removed IC2: L293D, st-microelectronics:L293D
- removed JP1: (no value), adafruit:PINHD-1X3
- removed U$5: LIPO-OUTLINE2000, SparkFun-Electromechanical:LIPO-OUTLINE2000
- removed U$6, U$7: MOTOR10MM, SparkFun-Electromechanical:MOTOR10MM
- added C2, C3: 0.1uF, adafruit:C-US050-024X044
- added JBAT, JCHG: (no value), SparkFun-Connectors:M02-JST-2-PTH-NO_SILK
- added JI2C: (no value), adafruit:PINHD-2X4
- added JIMU: PINHD-1X10, adafruit:PINHD-1X10
- added JM1, JM2: (no value), adafruit:PINHD-1X6
- added JNPX: (no value), adafruit:PINHD-1X3
- added M1, M2: MOTOR10MM, SparkFun-Electromechanical:MOTOR10MM
- added U3: L293D, st-microelectronics:L293D
- added U4: 7805T, adafruit:7805T
- C1: value (none) -> 10uF
- J1: device SparkFun-Connectors:M02-JST-2-PTH-NO_SILK -> adafruit:PINHD-1X3
- U1: device ESP32-DEVKITC:ESP32DEVKITC -> ESP32-DEVKITC (1):ESP32DEVKITC
- renumbered JP2 to J2, JP3 to J3, JP4 to J4
Connections:
- new net N$37: Q1.C, R2.1
- new net N$38: R15.2
- net GND: now also C2.2, J1.3, JBAT.2, JCHG.2, U1.GND@32, U1.GND@38, U3.GND1, U3.GND2, U3.GND3, U3.GND4, U4.GND; no longer IC2.GND1, IC2.GND2, IC2.GND3, IC2.GND4, J1.2, JP1.3
- net N$10: now also M1.+, U3.1Y; no longer IC2.1Y, U$6.+
- net N$11: now also M1.-, U3.2Y; no longer IC2.2Y, U$6.-
- net N$12: now also M2.-, U3.4Y; no longer IC2.4Y, U$7.-
- net N$13: now also M2.+, U3.3Y; no longer IC2.3Y, U$7.+
- net N$21: now also JCHG.1; no longer J1.1
- net N$23: now also J1.1; no longer JP1.1
- net N$4: now also U3.1A; no longer IC2.1A
- net N$5: now also U3.2A; no longer IC2.2A
- net N$6: now also U3.4A; no longer IC2.4A
- net N$7: now also U3.3A; no longer IC2.3A
- net N$8: now also U3.1-2EN; no longer IC2.1-2EN
- net N$9: now also U3.3-4EN; no longer IC2.3-4EN
- net V+: now also JBAT.1, U3.VCC2, U4.VI; no longer IC2.VCC2
- net VCC: now also C2.1, J1.2, U1.5V, U3.VCC1, U4.VO; no longer IC2.VCC1, JP1.2
Other:
- note added: "Licensing: Creative Commons ShareAlike 4.0 International - https://creativecommons.org/licenses/by-sa/4.0/ You are welcome to use this library for commercial purposes. For attribution, we ask that when you reproduce our board, you email us with a link."
- note added: "Remember to review CD4051 footprint & connections"
- moved on the sheet: C1, IC1, LED1, LED2, LED3, Q1, R1, R10, R11, R12, R13, R14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
