File: Project/PCB/MAIN/03/SWARMESH.brd (EAGLE design)
At the start: 75 x 75 mm, 48 parts, among them Q1 TIP122, U1 ESP32DEVKITC, U2 CD4051BEE4, U3 L293D, U4 L7805CV-DG, U5 TCRT5000L, U6 TCRT5000L

Commit message: update brd
Parts:
- removed GPIO17: (no value), adafruit:1X03
- moved T3 39.7 mm to (27.5, -14.7)
- moved T4 35.9 mm to (28.5, -5.47)
- moved T2 32.7 mm to (49.0, -6.74)
- moved T1 28.3 mm to (40.3, -13.3)
- moved C5 22.9 mm to (37.1, 46.7), turned to 90 degrees
- moved C2 9.42 mm to (21.3, 54.3)
- moved U6 2.56 mm to (38.4, 35.6)
- moved U5 1.59 mm to (38.4, 6.99)
- moved C6 1.59 mm to (60.0, 41.9)
- moved R15 1.59 mm to (17.8, 36.8)
- moved JP3 1.14 mm to (24.1, 70.5)
- moved JP4 1.14 mm to (12.7, 70.5)
- moved U1 1.14 mm to (26.0, 49.2)
- moved C4 0.64 mm to (18.4, 70.5)
- moved JP1 0.45 mm to (52.7, 70.8)
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Connections:
- removed net N$18: F1.2, S1.NC1
- new net N$2: F1.2, S1.C2
- new net N$3: BAT-.P$1, S1.C1
- net E1A: no longer GPIO17.1
- net GND: now also S1.NO1; no longer BAT-.P$1, GPIO17.3
- net V+: now also S1.NO2; no longer S1.NO1
- net VCC: no longer GPIO17.2
Routing:
- net GND: track 350.1 -> 485.6 mm
- net E2A: track 0.00 -> 100.5 mm
- net IO14: track 0.00 -> 83.0 mm
- net VCC: track 179.1 -> 257.7 mm
- net IO12: track 0.00 -> 65.6 mm
- net N$2: track 0.00 -> 60.7 mm
- net IR1: track 0.00 -> 60.5 mm
- net IR2: track 0.00 -> 56.8 mm
- net IO13: track 0.00 -> 50.3 mm
- net ADCMX: track 0.00 -> 49.4 mm
- net E1A: track 0.00 -> 49.0 mm
- net IO27: track 0.00 -> 48.5 mm
- net IRTX: track 0.00 -> 40.0 mm
- net N$9: track 0.00 -> 38.4 mm
- net N$3: track 0.00 -> 37.0 mm
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